File: Boards/Tractive System/IFE_Shutdown_2019/Shutdown_2019_v1.0/Shutdown_2019_v1.0.brd (EAGLE design)
At the start: 101.6 x 76.2 mm, 38 parts, among them IC1 LM555D, IC3 LM393D, Q1 IRLML6346PBF, Q2 IRLML6346PBF

Commit message: More shutdown work
Parts:
- added BMS1, BSPD, IMD: 3.3v BLUE, led:CHIPLED_0805
- added C1, C3, C4: 0.1uF, Capacitors:C0805
- added C14, C15, C16: 47uF, rcl:UD-6,3X5,8_NICHICON
- added D15, D2, D9: 1N914, Diodes:SOD323-F
- added D3, D5, D6: SMAJ12A, Diodes:DO-214AC
- added Q11, Q15, Q6: DMP3099L-7, TRANS:SOT23
- added Q16, Q3, Q5: DMN6140L-7, TRANS:SOT23
- added R1, R19, R24: 10k, Resistors:R0805
- added R11, R20, R23: 300, Resistors:R0805
- added R3, R5, R6: 100k, Resistors:R0805
- added R36: 1k, Resistors:R0805
- added U$10, U$12, U$13: PCN-112D3MHZ, Display_Custom:TH_SPST_PCN_D3M_TE_CONN
- U$4, U$7, U$8: value IRLL024ZPBF -> RT424012; device Display_Custom:SOT223 -> Display_Custom:TH_DPDT_GEN_PURPOSE_2.54
- moved BRAKE 61.6 mm to (3.81, 40.6)
- moved THROTTLE 61.0 mm to (10.2, 40.6)
- moved U$4 54.8 mm to (20.3, 61.0), turned to 90 degrees
- moved U$8 51.8 mm to (48.3, 61.0), turned to 90 degrees
- moved U$7 44.6 mm to (34.3, 61.0), turned to 90 degrees
- moved U$6 36.4 mm to (78.7, 71.1), turned to 180 degrees
- moved PWR 24.1 mm to (96.5, 45.7)
- moved U$3 19.0 mm to (96.5, 35.6)
- moved U$5 17.8 mm to (61.0, 5.08)
- moved CAN 16.5 mm to (73.7, 5.08)
- moved HALL_SENSE 6.35 mm to (96.5, 22.9)
- moved U$2 6.35 mm to (5.08, 55.9)
- moved U$1 6.35 mm to (5.08, 64.8)
Connections:
- new net BMS1_FAULT_INDICATOR: C15.+, D9.C, R20.1, U$7.21, U$7.A1
- new net BSPD_FAULT_INDICATOR: C16.+, D2.C, R11.1, U$4.21, U$4.A1
- new net FAULT_2_BMS: Q3.1, R1.2
- new net FAULT_3_BMS2_IN: C3.1, D5.C, R5.2
- new net FAULT_4_IMD_IN: C4.1, D6.C, Q16.1, R24.2, R6.2
- new net FAULT_RESET: Q11.1, Q15.1, Q6.1, R36.2
- new net IMD_FAULT_INDICATOR: C14.+, D15.C, R23.1, U$8.21, U$8.A1
- new net N$1: C15.-, D9.A, Q3.3, U$7.A2
- new net N$27: U$4.14, U$7.11
- new net N$28: Q6.3, U$4.22
- new net N$31: U$7.14, U$8.11
- new net N$32: C16.-, D2.A, Q5.3, U$4.A2
- new net N$34: BMS1.A, R20.2
- new net N$35: Q11.3, U$7.22
- new net N$42: IMD.A, R23.2
- new net N$43: Q15.3, U$8.22
- new net N$44: C14.-, D15.A, Q16.3, U$8.A2
- new net N$8: BSPD.A, R11.2
- net +12V: now also Q11.2, Q15.2, Q6.2, R36.1, U$4.24, U$7.24, U$8.24
- net AIR_IN: now also U$4.11
- net AIR_OUT: now also U$8.14
- net FAULT_1_BSPD_IN: now also C1.1, D3.C, Q5.1, R19.2, R3.2
- net GND: now also BMS1.C, BSPD.C, C1.2, C3.2, C4.2, D3.A, D5.A, D6.A, IMD.C, Q16.2, Q3.2, Q5.2, R1.1, R19.1, R24.1, R3.1, R5.1, R6.1

Commit message: Adding circuitry to shutdown, relay drivers
Parts:
- removed U$10, U$12, U$13: PCN-112D3MHZ, Display_Custom:TH_SPST_PCN_D3M_TE_CONN
- removed U$4, U$7, U$8: RT424012, Display_Custom:TH_DPDT_GEN_PURPOSE_2.54
- added H1, H2, H3, H4: MOUNT-PAD-ROUND3.0, holes:3,0-PAD
- added Q4, Q7, Q8: DMN6140L-7, TRANS:SOT23
- added R2, R4, R7: 10k, Resistors:R0805
- added R_APPS, R_BTSF, R_RTD: PCN-112D3MHZ, Display_Custom:TH_SPST_PCN_D3M_TE_CONN
- added R_BMS, R_BSPD, R_IMD: RT424012, Display_Custom:TH_DPDT_GEN_PURPOSE_2.54
- added U1, U2: STM32F103CBT6, ST Microelctronics_By_element14_Batch_1:QFP50P900X900X160-48N
- moved BSPD 81.7 mm to (20.3, 38.1), turned to 90 degrees
- moved IC3 67.3 mm to (6.35, 30.5)
- moved IC1 40.6 mm to (6.35, 19.1)
- moved CAN 17.8 mm to (55.9, 5.08)
- moved U$5 15.2 mm to (45.7, 5.08)
- moved TSAL 3.81 mm to (22.9, 5.08)
- moved U$2 1.27 mm to (5.08, 54.6)
- moved U$6 1.27 mm to (77.5, 71.1)
- renumbered BMS1 to BMS
Connections:
- new net APPS_EN: Q4.1, R2.2
- new net BTSF_EN: Q7.1, R4.2
- new net N$12: R_BTSF.3, R_RTD.4
- new net N$13: R_APPS.3, R_BTSF.4
- new net N$2: Q4.3, R_APPS.2
- new net N$4: Q7.3, R_BTSF.2
- new net N$9: Q8.3, R_RTD.2
- new net PA11: U1.32, U2.32
- new net PRECHARGE_COMPLETE: U$3.3
- new net RTDS-: TSAL.3
- new net RTD_EN: Q8.1, R7.2
- new net VDDA: U1.9, U2.9
- new net VDD_2: U1.36, U2.36
- new net VDD_3: U1.48, U2.48
- net +12V: now also R_BMS.24, R_BSPD.24, R_IMD.24; no longer U$4.24, U$7.24, U$8.24
- net AIR_IN: now also R_BSPD.11; no longer U$4.11
- net AIR_OUT: now also R_IMD.14; no longer U$8.14
- net BMS1_FAULT_INDICATOR: now also R_BMS.21, R_BMS.A1; no longer U$7.21, U$7.A1
- net BSPD_FAULT_INDICATOR: now also R_BSPD.21, R_BSPD.A1; no longer U$4.21, U$4.A1
- net ENABLE_IN: now also R_APPS.4
- net ENABLE_OUT: now also R_RTD.3
- net GND: now also H1.B3,0, H2.B3,0, H3.B3,0, H4.B3,0, Q4.2, Q7.2, Q8.2, R2.1, R4.1, R7.1
- net IMD_FAULT_INDICATOR: now also R_IMD.21, R_IMD.A1; no longer U$8.21, U$8.A1
- net N$1: now also R_BMS.A2; no longer U$7.A2
- net N$27: now also R_BMS.11, R_BSPD.14; no longer U$4.14, U$7.11
- net N$28: now also R_BSPD.22; no longer U$4.22
- net N$31: now also R_BMS.14, R_IMD.11; no longer U$7.14, U$8.11
- net N$32: now also R_BSPD.A2; no longer U$4.A2
- net N$35: now also R_BMS.22; no longer U$7.22
- net N$43: now also R_IMD.22; no longer U$8.22
- net N$44: now also R_IMD.A2; no longer U$8.A2

Commit message: Safety board cleanup
Parts:
- removed !BSPD_FAULT, !CONFLICT, BCO, BTH, TCO, TTH: TPTP09R, testpad:TP09R
- removed BMS, BSPD, IMD: 3.3v BLUE, led:CHIPLED_0805
- removed BRAKE, THROTTLE: RTRIM3249W, Resistors:RTRIM3299W
- removed C18: 10uF, Capacitors:C0805
- removed C19: 0.01uF, Capacitors:C0805
- removed C24: 0.1uF, Capacitors:C0805
- removed IC1: LM555D, bspd2:SO08
- removed IC3: LM393D, IC's:SO08
- removed Q1, Q2: IRLML6346PBF, TRANS:SOT23
- removed R13: 50k, Resistors:R0805
- removed R14, R19, R24, R33, R38, R39, R40: 10k, Resistors:R0805
- removed R20, R23: 300, Resistors:R0805
- removed R3, R6, R9: 100k, Resistors:R0805
- removed R36: 1k, Resistors:R0805
- removed U$11: SN74LVC1G04DBVR, Display_Custom:SOT23-5L
- removed U$9: SN74LVC1G132DBVR, Display_Custom:SOT23-5L
- removed U2: STM32F103CBT6, ST Microelctronics_By_element14_Batch_1:QFP50P900X900X160-48N
- added BRAKE1, THROTTLE1: RTRIM3249W, Resistors:RTRIM3299W
- added BTH1, TTH1: TPTP09R, testpad:TP09R
- added C5, C6, C7: 0.1u, resistor:C0603
- added D1, D4, D7: BLUE, SparkFun-LED:LED-0603
- added Q12, Q13, Q14, Q17: IRLML6346PBF, TRANS:SOT23
- added R15, R21, R22: 900, resistor:R0603
- added R16, R17, R18, R25: 10k, resistor:R0603
- C1: value 0.1uF -> 0.1u; device Capacitors:C0805 -> resistor:C0603
- C3, C4: value 0.1uF -> 3u; device Capacitors:C0805 -> resistor:C0603
- D3, D5, D6: value SMAJ12A -> 1N914; device Diodes:DO-214AC -> Diodes:SOD323-F
- R1: value 10k -> 100k; device Resistors:R0805 -> resistor:R0603
- R10: value 1k -> 10k; device Resistors:R0805 -> resistor:R0603
- R11: value 300 -> 100k; device Resistors:R0805 -> resistor:R0603
- R5: value 100k -> 10k; device Resistors:R0805 -> resistor:R0603
- R8: device Resistors:R0805 -> resistor:R0603
- moved Q8 179.3 mm to (55.9, 62.2), flipped to the bottom, turned to 270 degrees
- moved R2 174.5 mm to (121.9, 33.0)
- moved R4 174.5 mm to (121.9, 17.8)
- moved R7 174.5 mm to (121.9, 2.54)
- moved Q7 167.6 mm to (62.2, 62.2), flipped to the bottom, turned to 270 degrees
- moved Q4 156.9 mm to (68.6, 62.2), flipped to the bottom, turned to 270 degrees
- moved R11 138.8 mm to (-24.1, 19.1)
- moved D2 127.3 mm to (17.8, 49.5), flipped to the bottom, turned to 180 degrees
- moved D9 124.4 mm to (31.8, 49.5), flipped to the bottom, turned to 180 degrees
- moved C4 124.3 mm to (-21.6, 14.0)
- moved C3 122.3 mm to (-25.4, 14.0)
- moved D15 118.4 mm to (45.7, 49.5), flipped to the bottom, turned to 180 degrees
- moved Q15 118.2 mm to (45.7, 62.2), flipped to the bottom, turned to 180 degrees
- moved Q6 115.0 mm to (17.8, 62.2), flipped to the bottom, turned to 180 degrees
- moved Q11 114.6 mm to (31.8, 62.2), flipped to the bottom, turned to 180 degrees
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Connections:
- removed net !CONFLICT: !CONFLICT.TP, IC1.2, R8.2, U$9.4
- removed net BSPD_FAULT: IC1.3, U$11.2
- removed net FAULT_1_BSPD_IN: C1.1, D3.C, Q2.3, Q5.1, R10.2, R19.2, R3.2
- removed net FAULT_2_BMS: Q3.1, R1.2
- removed net FAULT_3_BMS2_IN: C3.1, D5.C, R5.2
- removed net FAULT_4_IMD_IN: C4.1, D6.C, Q16.1, R24.2, R6.2
- removed net N$15: Q1.3, Q2.1, R9.2
- removed net N$16: IC3.6, THROTTLE.2, TTH.TP
- removed net N$3: IC3.7, R39.1, TCO.TP, U$9.1
- removed net N$5: BCO.TP, IC3.1, R38.1, U$9.2
- removed net N$6: BRAKE.2, BTH.TP, IC3.2
- new net BRAKE_TH: BRAKE1.2, BTH1.TP
- new net BSPD_FAULT_INDICATOR1: D3.C
- new net BSPD_FAULT_INDICATOR2: D5.C
- new net BSPD_FAULT_INDICATOR3: D6.C
- new net FAULT_BMS: C6.1, Q3.1, R17.2
- new net FAULT_BSPD: C7.1, Q12.3, Q14.3, Q17.3, Q5.1, R16.2, R5.1
- new net FAULT_IMD: C5.1, Q16.1, R18.2
- new net THROTTLE_TH: THROTTLE1.2, TTH1.TP
- net +12V: now also R25.2, R5.2; no longer R10.1, R36.1, R9.1
- net +5V: now also BRAKE1.1, C1.1, R1.2, R10.2, R11.2, R8.2, THROTTLE1.1; no longer BRAKE.1, C24.1, IC1.4, IC1.8, IC3.8, R13.2, R14.2, R33.2, R38.2, R39.2, R40.1, R8.1, THROTTLE.1, U$11.5, U$9.5
- net BMS1_FAULT_INDICATOR: now also R22.1; no longer R20.1
- net BRAKE_IN: now also R10.1; no longer IC3.3, R33.1
- net BSPD_FAULT_INDICATOR: now also R15.1; no longer R11.1
- net CURRENT_IN: now also R8.1; no longer IC3.5, R14.1
- net FAULT_RESET: now also R25.1; no longer R36.2
- net GND: now also BRAKE1.3, C14.-, C15.-, C16.-, C5.2, C6.2, C7.2, D1.C, D4.C, D7.C, Q13.2, Q14.2, Q17.2, R16.1, R17.1, R18.1, THROTTLE1.3; no longer BMS.C, BRAKE.3, BSPD.C, C18.2, C19.2, C24.2, D3.A, D5.A, D6.A, IC1.1, IC3.4, IMD.C, Q1.2, Q2.2, R1.1, R19.1, R24.1, R3.1, R5.1, R6.1, THROTTLE.3, U$11.3, U$9.3
- net IMD_FAULT_INDICATOR: now also R21.1; no longer R23.1
- net N$1: no longer C15.-
- net N$10: now also D5.A, Q7.3, R_BTSF.2; no longer C18.1, IC1.6, IC1.7, R13.1
- net N$11: now also D6.A, Q8.3, R_RTD.2; no longer C19.1, IC1.5
- net N$2: now also C3.1, R11.1; no longer Q4.3, R_APPS.2
- net N$32: no longer C16.-
- net N$34: now also D4.A, R22.2; no longer BMS.A, R20.2
- net N$4: now also C4.1, R1.1; no longer Q7.3, R_BTSF.2
- net N$42: now also D1.A, R21.2; no longer IMD.A, R23.2
- net N$44: no longer C14.-
- net N$7: now also D3.A, Q4.3, R_APPS.2; no longer !BSPD_FAULT.TP, Q1.1, R40.2, U$11.4
- net N$8: now also D7.A, R15.2; no longer BSPD.A, R11.2
- net N$9: now also Q12.2, Q13.3; no longer Q8.3, R_RTD.2
- net PA11: no longer U2.32
- net VDDA: no longer U2.9
- net VDD_2: no longer U2.36
- net VDD_3: no longer U2.48
Other:
- board size 101.6 x 76.2 mm -> 88.9 x 76.2 mm
