File: Boards/Tractive System/IFE_Shutdown_2019/Shutdown_2019_v1.0_UNROUTED/Shutdown_2019_v1.0.brd (EAGLE design)
At the start: 88.9 x 76.2 mm, 194 parts, among them Q1 DMN6140L-7, Q10 DMN6140L-7, Q11 DMP3099L-7, Q12 IRLML6346PBF, Q13 IRLML6346PBF, Q14 IRLML6346PBF, Q15 DMP3099L-7, Q16 DMN6140L-7, Q17 IRLML6346PBF, Q18 DMN6140L-7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

Commit message: nearly done with routing
Parts:
- added R45: 10k, rcl:R0603
- moved C17 7.37 mm to (72.4, 2.54)
- moved R19 7.37 mm to (69.8, 2.54), turned to 90 degrees
- moved C18 7.37 mm to (72.4, 10.2), turned to 270 degrees
- moved R20 7.37 mm to (69.8, 10.2), turned to 270 degrees
- moved R11 6.35 mm to (21.6, 37.8)
- moved R39 5.08 mm to (16.0, 37.8)
- moved R43 0.76 mm to (18.0, 37.8)
- moved C15 0.51 mm to (60.2, 30.0)
- moved C19 0.51 mm to (62.2, 30.0)
- moved C16 0.51 mm to (29.0, 29.5)
- moved C20 0.51 mm to (29.0, 31.5)
- moved R40 0.51 mm to (23.6, 37.8)
- moved D9 0.25 mm to (30.7, 62.5)
- moved R23 0.25 mm to (55.9, 64.0)
Connections:
- net +5V: now also R45.2
- net CANH: now also CAN.1; no longer CAN.2
- net CANL: now also CAN.2; no longer CAN.1
- net HALL_FL_F: now also U2.25; no longer U2.11
- net HALL_FR_F: now also U2.26; no longer U2.10
- net HALL_RL_F: now also U2.27; no longer U2.12
- net HALL_RR_F: now also U2.28; no longer U2.13
- net THROTTLE_OUT: now also R45.1
Routing:
- net +5V: track 172.1 -> 0.00 mm, vias 22 -> 0
- net +3V3: track 163.4 -> 0.00 mm, vias 10 -> 0
- net +12V: track 161.4 -> 0.00 mm, vias 4 -> 0
- net FAULT_BSPD_STATUS_3_3: track 70.7 -> 0.00 mm, vias 5 -> 0
- net RTDS_EN: track 62.8 -> 0.00 mm, vias 4 -> 0
- net FAULT_BMS_STATUS_3_3: track 57.2 -> 0.00 mm, vias 3 -> 0
- net FAULT_IMD_STATUS_3_3: track 48.9 -> 0.00 mm, vias 3 -> 0
- net RTD_EN: track 47.2 -> 0.00 mm, vias 2 -> 0
- net BRAKE_PRESSURE_F_3_3: track 46.3 -> 0.00 mm, vias 4 -> 0
- net HV_CONNECTED_3_3: track 45.8 -> 0.00 mm
- net AIR_OUT: track 45.8 -> 0.00 mm
- net BTSF_EN: track 44.4 -> 0.00 mm, vias 2 -> 0
- net APPS_EN: track 43.9 -> 0.00 mm
- net FAULT_RESET_F: track 43.5 -> 0.00 mm, vias 3 -> 0
- net FAULT_IMD: track 39.0 -> 0.00 mm, vias 1 -> 0
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