File: Boards/Tractive System/IFE_DASH_2019/DASH_BOARD_V_2.0.brd (EAGLE design)
At the start: 160 x 100 mm, 77 parts, among them IC1 STM32F10XCXT6

Commit message: more tweaks
Parts:
- moved R7 46.7 mm to (71.1, 16.5)
- moved R3 37.0 mm to (83.8, 8.89)
- moved R1 35.8 mm to (71.1, 22.9)
- moved S1 34.5 mm to (83.8, 20.3)
- moved D5 24.7 mm to (67.3, 16.5), turned to 90 degrees
- moved R6 23.7 mm to (56.3, 16.5)
- moved D4 18.1 mm to (67.3, 22.9), turned to 90 degrees
- moved D3 17.6 mm to (67.3, 19.8)
- moved R8 17.1 mm to (56.2, 23.1)
- moved D1 16.2 mm to (68.6, 11.4), turned to 270 degrees
- moved L4 8.98 mm to (11.4, 21.6), turned to 0 degrees
- moved R10 8.69 mm to (56.1, 19.8)
- moved R2 7.84 mm to (71.1, 19.7), turned to 0 degrees
- moved C2 7.76 mm to (18.5, 23.4)
- moved C5 7.66 mm to (12.3, 27.6), turned to 90 degrees
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Connections:
- net PHONE_RX/U_TX: now also U$10.3; no longer U$10.4
- net PHONE_TX/U_RX: now also U$10.4; no longer U$10.3
Routing:
- net +5V: track 0.00 -> 139.7 mm, vias 0 -> 4
- net PWR: track 0.00 -> 37.6 mm
- net ENABLE: track 0.00 -> 33.4 mm
- net +3V3: track 0.00 -> 33.3 mm, vias 0 -> 3
- net N$8: track 0.00 -> 21.5 mm
- net N$12: track 0.00 -> 20.8 mm, vias 0 -> 1
- net N$3: track 0.00 -> 20.3 mm
- net CAN_H: track 0.00 -> 20.3 mm
- net CAN_L: track 0.00 -> 18.8 mm
- net PHONE_RX/U_TX: track 0.00 -> 16.6 mm
- net PHONE_TX/U_RX: track 0.00 -> 13.1 mm
- net N$6: track 0.00 -> 12.1 mm
- net PHONE_POWER: track 0.00 -> 11.6 mm
- net SWCLK: track 0.00 -> 10.1 mm, vias 0 -> 1
- net SWDIO: track 0.00 -> 9.97 mm
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
Commit message: more routing
Parts:
- moved R7 1.16 mm to (70.9, 15.4)
- moved D5 1.15 mm to (67.2, 15.4)
- moved D12 0.81 mm to (29.6, 28.9)
- moved D4 0.77 mm to (67.4, 23.6)
- moved R1 0.66 mm to (71.1, 23.5)
- moved D3 0.45 mm to (67.1, 19.4)
- moved R2 0.44 mm to (70.9, 19.3)
- moved R13 0.33 mm to (31.4, 28.9)
- moved R33 0.10 mm to (56.6, 47.0), turned to 90 degrees
- turned R37 to 300 degrees
Connections:
- net DRS_VALUE: now also IC1.10; no longer IC1.18
Routing:
- net DRS_VALUE: track 0.00 -> 60.2 mm
- net CURRENT_VALUE: track 0.00 -> 51.8 mm
- net TC_VALUE: track 0.00 -> 38.2 mm
- net +3V3: track 33.3 -> 59.3 mm
- net RESET: track 0.00 -> 22.1 mm, vias 0 -> 1
- net +5V: track 139.7 -> 158.1 mm
- net CAN_RX/STM_TX: track 0.00 -> 15.9 mm
- net CAN_TX/STM_RX: track 0.00 -> 12.9 mm
- net DASH_PRE_DONE: track 0.00 -> 10.6 mm, vias 0 -> 1
- net DASH_POWER_ON: track 0.00 -> 8.33 mm, vias 0 -> 1
- net N$36: track 0.00 -> 7.82 mm
- net N$14: track 0.00 -> 7.78 mm
- net N$23: track 0.00 -> 7.61 mm
- net N$18: track 0.00 -> 7.53 mm
- net N$30: track 0.00 -> 7.47 mm
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Other:
- board text added: "BLUE: PRECHARGEING"
- board text added: "BMS FAULT"
- board text added: "BSPD FAULT"
- board text added: "GREEN: PRECHARE DONE"
- board text added: "IMD FAULT"
- board text added: "RED: LV ON"

Commit message: v2 done
Parts:
- removed U$11, U$12: DMN2300U, Display_Custom:SOT23
- added C1, C3, C4, C6: 0.1u, rcl:C0805K
- added CUSTOM_POT: SWITCH_ROTARY_1X10KIT, Testing:ROTARY_SWITCH_1X10_KIT
- added D6: DRS_BLUE, SparkFun-LED:LED-0603
- added D7: TC_BLUE, SparkFun-LED:LED-0603
- added Q1, Q2, Q6: DMP3099L-7, TRANS:SOT23
- added R4, R47, R48, R49, R5, R50, R51, R52, R53, R54, R55, R9: 10k, resistor:R0805
- added R56: 1k, resistor:R0805
- added R57, R58: 330, resistor:R0805
- added U$7: DMN2300U, Display_Custom:SOT23
- R1, R2, R7: value 10k -> 330
- R10: value 1k -> 85
- R13, R14: value (none) -> 330
- R6: value 1k -> 140
- R8: value 1k -> 90
- moved R3 31.8 mm to (83.8, 40.6), turned to 0 degrees
- moved U$9 20.8 mm to (38.1, 33.0), flipped to the top
- moved S1 17.7 mm to (90.2, 36.8), turned to 180 degrees
- moved D1 12.7 mm to (61.0, 21.6), turned to 90 degrees
- moved R1 11.9 mm to (62.3, 15.4), flipped to the bottom
- moved R2 11.1 mm to (63.6, 11.0), flipped to the bottom
- moved R7 11.1 mm to (63.5, 7.11), flipped to the bottom
- moved D4 8.13 mm to (62.3, 17.3)
- moved D3 8.02 mm to (62.3, 12.9)
- moved D5 7.27 mm to (63.5, 9.12)
- moved H6 5.79 mm to (7.14, 67.6), turned to 180 degrees
- moved R30 5.77 mm to (45.9, 65.3)
- moved DRS_POT 5.77 mm to (18.0, 52.6)
- moved R26 5.77 mm to (34.7, 46.5)
- moved R27 5.77 mm to (33.5, 52.6)
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Connections:
- removed net CAN_RX/STM_TX: IC1.33, U$6.4
- removed net CAN_TX/STM_RX: IC1.32, U$6.1
- removed net DASH_POWER_ON: IC1.20, U$9.1
- removed net DASH_PRE_DONE: IC1.22, U$12.1
- removed net DASH_PRE_STARTED: IC1.21, U$11.1
- new net CAN_RX: IC1.32, U$6.4
- new net CAN_TX: IC1.33, U$6.1
- new net CUSTOM_VALUE: CUSTOM_POT.COMMON, IC1.11
- new net DRS_: D6.A, R57.1
- new net DRS_LED: IC1.29, U$7.1
- new net N$1: Q6.3, R6.2
- new net N$24: Q1.3, R10.2
- new net N$27: Q2.3, R8.2
- new net N$34: CUSTOM_POT.2, R47.2, R48.1
- new net N$35: CUSTOM_POT.3, R48.2, R49.2
- new net N$45: CUSTOM_POT.4, R49.1, R50.2
- new net N$46: CUSTOM_POT.5, R50.1, R51.2
- new net N$47: CUSTOM_POT.6, R51.1, R52.2
- new net N$48: CUSTOM_POT.7, R52.1, R53.2
- new net N$49: CUSTOM_POT.8, R53.1, R54.2
- new net N$50: CUSTOM_POT.9, R54.1, R55.2
- new net N$51: CUSTOM_POT.1, R47.1, R56.1
- new net N$52: D6.C, U$7.3
- new net N$53: D7.C, U$9.3
- new net RGB_BLUE: IC1.21, Q1.1, R5.2
- new net RGB_GREEN: IC1.22, Q2.1, R9.2
- new net RGB_RED: IC1.20, Q6.1, R4.2
- new net TC_: D7.A, R58.1
- new net TC_LED: IC1.30, U$9.1
- net +3V3: now also C1.1, C3.1, C4.1, C6.1
- net +5V: now also Q1.2, Q2.2, Q6.2, R4.1, R5.1, R56.2, R57.2, R58.2, R9.1; no longer R10.2, R6.2, R8.2
- net GND: now also C1.2, C3.2, C4.2, C6.2, CUSTOM_POT.10, R55.1, U$7.2; no longer U$11.2, U$12.2
- net N$15: no longer U$11.3
- net N$16: no longer U$9.3
- net N$5: no longer U$12.3
Routing:
- net +5V: track 158.1 -> 291.2 mm, vias 4 -> 6
- net CUSTOM_VALUE: track 0.00 -> 64.2 mm
- net GND: track 0.00 -> 51.6 mm, vias 0 -> 10
- net DRS_LED: track 0.00 -> 35.1 mm, vias 0 -> 2
- net ENABLE: track 33.4 -> 64.2 mm
- net +3V3: track 59.3 -> 88.1 mm, vias 3 -> 4
- net CAN_RX: track 0.00 -> 17.8 mm
- net CAN_RX/STM_TX: track 15.9 -> 0.00 mm
- net CURRENT_VALUE: track 51.8 -> 66.8 mm
- net RGB_BLUE: track 0.00 -> 14.0 mm, vias 0 -> 1
- net RGB_GREEN: track 0.00 -> 13.9 mm, vias 0 -> 2
- net RGB_RED: track 0.00 -> 13.0 mm, vias 0 -> 1
- net CAN_TX/STM_RX: track 12.9 -> 0.00 mm
- net CAN_TX: track 0.00 -> 11.6 mm
- net DASH_PRE_DONE: track 10.6 -> 0.00 mm, vias 1 -> 0
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- added copper zone on layer 1, net GND
- added copper zone on layer 16, net GND
Other:
- board size 160 x 100 mm -> 99.1 x 74.6 mm
- board text added: "1"
- board text added: "10"
- board text added: "CURRENT POT"
- board text added: "DRS POT"
- board text added: "Dashboard v2.0 Apollo 2019"
- board text added: "Illini Formula Electric"
- board text added: "Nick Tuczak"
- board text added: "TC POT"
- board text removed: "BLUE: PRECHARGEING"
- board text removed: "GREEN: PRECHARE DONE"
- board text removed: "RED: LV ON"

Commit message: final revisions for 2
Connections:
- net GND: now also IC1.20
- net RGB_RED: now also IC1.18; no longer IC1.20
Routing:
- net GND: track 51.6 -> 57.4 mm, vias 10 -> 11
Changed lines of the file:
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@@
 <wire x1="36.7538" y1="28.1178" x2="35.7006" y2="28.1178" width="0.254" layer="1"/>
 <wire x1="35.7006" y1="28.1178" x2="35.687" y2="28.1314" width="0.254" layer="1"/>
+<contactref element="IC1" pad="20"/>
+<via x="48.2092" y="18.2118" extent="1-16" drill="0.2"/>
+<wire x1="48.2092" y1="18.2118" x2="47.6409375" y2="18.2118" width="0.254" layer="1"/>
+<wire x1="47.6409375" y1="18.2118" x2="47.4163375" y2="18.4364" width="0.254" layer="1"/>
+<wire x1="47.4163375" y1="18.4364" x2="44.1492" y2="18.4364" width="0.254" layer="1"/>
+<wire x1="44.1492" y1="18.4364" x2="44.069" y2="18.5166" width="0.254" layer="1"/>
+<wire x1="44.069" y1="18.5166" x2="42.6134" y2="18.5166" width="0.254" layer="1"/>
+<wire x1="42.6134" y1="18.5166" x2="42.6" y2="18.53" width="0.254" layer="1"/>
 </signal>
 <signal name="+3V3">
@@
 <contactref element="CURRENT_POT" pad="COMMON"/>
 <contactref element="IC1" pad="19"/>
-<wire x1="75.1078" y1="58.078" x2="75.1078" y2="50.0634" width="0.254" layer="1"/>
-<wire x1="75.1078" y1="50.0634" x2="75.1078" y2="38.2778" width="0.254" layer="1"/>
+<wire x1="75.1078" y1="58.078" x2="75.1078" y2="38.2778" width="0.254" layer="1"/>
 <wire x1="75.1078" y1="38.2778" x2="63.5" y2="26.67" width="0.254" layer="1"/>
-<wire x1="63.5" y1="26.67" x2="63.5" y2="20.32" width="0.254" layer="1"/>
-<wire x1="63.5" y1="20.32" x2="63.5" y2="19.3802" width="0.254" layer="1"/>
+<wire x1="63.5" y1="26.67" x2="63.5" y2="19.3802" width="0.254" layer="1"/>
 <wire x1="63.5" y1="19.3802" x2="62.8904" y2="18.7706" width="0.254" layer="1"/>
 <wire x1="62.8904" y1="18.7706" x2="60.8584" y2="18.7706" width="0.254" layer="1"/>
 <wire x1="60.8584" y1="18.7706" x2="57.9374" y2="15.8496" width="0.254" layer="1"/>
-<wire x1="57.9374" y1="15.8496" x2="57.15" y2="15.8496" width="0.254" layer="1"/>
-<wire x1="57.15" y1="15.8496" x2="56.7436" y2="15.8496" width="0.254" layer="1"/>
-<wire x1="56.7436" y1="15.8496" x2="49.4284" y2="15.8496" width="0.254" layer="1"/>
-<wire x1="49.4284" y1="15.8496" x2="48.0822" y2="17.1958" width="0.254" layer="1"/>
-<wire x1="48.0822" y1="17.1958" x2="44.9326" y2="17.1958" width="0.254" layer="1"/>
-<wire x1="44.9326" y1="17.1958" x2="44.9072" y2="17.1704" width="0.254" layer="1"/>
-<wire x1="44.9072" y1="17.1704" x2="43.934" y2="17.1704" width="0.254" layer="1"/>
-<wire x1="43.934" y1="17.1704" x2="43.3794" y2="17.725" width="0.254" layer="1"/>
-<wire x1="43.3794" y1="17.725" x2="43.3794" y2="17.74573125" width="0.254" layer="1"/>
-<wire x1="43.3794" y1="17.74573125" x2="43.09513125" y2="18.03" width="0.254" layer="1"/>
-<wire x1="43.09513125" y1="18.03" x2="42.6" y2="18.03" width="0.254" layer="1"/>
+<wire x1="57.9374" y1="15.8496" x2="49.4284" y2="15.8496" width="0.254" layer="1"/>
+<wire x1="49.4284" y1="15.8496" x2="48.514" y2="16.764" width="0.254" layer="1"/>
+<wire x1="48.514" y1="16.764" x2="48.0822" y2="17.1958" width="0.254" layer="1"/>
+<wire x1="42.6" y1="18.03" x2="47.248" y2="18.03" width="0.254" layer="1"/>
+<wire x1="47.248" y1="18.03" x2="48.0822" y2="17.1958" width="0.254" layer="1"/>
 </signal>
 <signal name="N$25">
@@
 <contactref element="Q6" pad="1"/>
 <contactref element="R4" pad="2"/>
-<contactref element="IC1" pad="20"/>
-<wire x1="42.6" y1="18.53" x2="45.097" y2="18.53" width="0.254" layer="1"/>
-<wire x1="45.097" y1="18.53" x2="45.5168" y2="18.1102" width="0.254" layer="1"/>
-<via x="45.5168" y="18.1102" extent="1-16" drill="0.35"/>
-<wire x1="45.5168" y1="18.1102" x2="46.4668" y2="17.1602" width="0.254" layer="16"/>
-<wire x1="46.4668" y1="17.1602" x2="49.4714" y2="17.1602" width="0.254" layer="16"/>
+<wire x1="44.7396" y1="17.1602" x2="49.4714" y2="17.1602" width="0.254" layer="16"/>
 <wire x1="49.4714" y1="17.1602" x2="50.3248" y2="16.3068" width="0.254" layer="16"/>
 <wire x1="50.3248" y1="16.3068" x2="54.6506" y2="16.3068" width="0.254" layer="16"/>
+<wire x1="44.7396" y1="17.1602" x2="44.6024" y2="17.2974" width="0.254" layer="16"/>
+<via x="44.6024" y="17.2974" extent="1-16" drill="0.35"/>
+<contactref element="IC1" pad="18"/>
+<wire x1="42.6" y1="17.53" x2="44.3698" y2="17.53" width="0.254" layer="1"/>
+<wire x1="44.3698" y1="17.53" x2="44.6024" y2="17.2974" width="0.254" layer="1"/>
 </signal>
 <signal name="RGB_BLUE">
