File: Boards/Tractive System/IFE_DASH_2019/DASH_BOARD_V_2.0.sch (EAGLE design)
At the start: 34 parts, among them IC1 STM32F10XCXT6

Commit message: dash v_2 cleanup
Parts:
- removed I/O1: MINIFIT_JR_5566-10, Display_Custom:MINIFIT_JR_5566-10
- removed POWER: 3.3V Blue, led:LEDSML0805
- removed R4, R9: 10k, resistor:R-US_R0805
- removed R5: 330, rcl:R-US_R0805
- removed U$7: MINIFIT_JR_5566-04, Display_Custom:MINIFIT_JR_5566-04
- added C2: 220u, rcl:CPOL-USE2.5-7
- added CURRENT_POT, DRS_POT, TC_POT: SWITCH_ROTARY_1X10KIT, Testing:SWITCH_ROTARY_1X10KIT
- added D1: XZM2CRKM2DGFBB45SCCB, SparkFun-LED:SUNLEDSMD1
- added D11, D12: GREEN, SparkFun-LED:LED-GREEN0603
- added D3: BSPD_RED, SparkFun-LED:LED-GREEN0603
- added D4: IMD_RED, SparkFun-LED:LED-GREEN0603
- added D5: BMS_RED, SparkFun-LED:LED-GREEN0603
- added FUSE: MINI297-3568, Fuse:MINI297-3568
- added FUSE1: 10 amp phone fuse, Fuse:MINI297-3568
- added L4: 10u, microbuilder:INDUCTORNR5040
- added R13, R14: (no value), rcl:R-US_R0603
- added R15, R17, R19, R20, R21, R22, R23, R24, R25, R26, R27, R28, R29, R30, R31, R32, R33, R34, R35, R36, R37, R38, R39, R40, R41, R42, R43: 10k, resistor:R-US_R0805
- added R44, R45, R46: 1k, resistor:R-US_R0805
- added S1: (no value), switch:320-916
- added U$10: MINIFIT_JR_5566-04, Display_Custom:MINIFIT_JR_5566-04
- added U$11, U$12: DMN2300U, Display_Custom:DMN2300U
- R10, R6, R8: value 10k -> 1k
- U$5: value DMN2300U -> MINIFIT_JR_5566-02; device Display_Custom:DMN2300U -> Display_Custom:MINIFIT_JR_5566-02
- U$9: value MINIFIT_JR_5566-02 -> DMN2300U; device Display_Custom:MINIFIT_JR_5566-02 -> Display_Custom:DMN2300U
Connections:
- removed net +12V: U$8.1
- removed net CURRENT_LIMIT: IC1PORTA_L.PA2, R3.1, U$7.1
- removed net N$1: POWER.A, R5.1
- removed net PRECHARGE_COMPLETE: IC1PORTA_L.PA7, U$5.G
- removed net PRECHARGE_LED_ON: I/O1.7, R4.1, U$5.D
- removed net TC_ON/OFF: IC1PORTA_L.PA3, R9.1, U$7.2
- new net CURRENT_VALUE: CURRENT_POT.COMMON, IC1PORTB_L.PB1
- new net DASH_POWER_ON: IC1PORTB_L.PB2, U$9.G
- new net DASH_PRE_DONE: IC1PORTB_H.PB11, U$12.G
- new net DASH_PRE_STARTED: IC1PORTB_H.PB10, U$11.G
- new net DRS_VALUE: DRS_POT.COMMON, IC1PORTB_L.PB0
- new net ENABLE: S1.P, U$5.1
- new net N$10: D12.C, R13.2
- new net N$11: D11.C, R14.2
- new net N$12: D3.C, U$1.D
- new net N$13: CURRENT_POT.3, R17.2, R19.2
- new net N$14: CURRENT_POT.1, R15.1, R44.1
- new net N$15: D1.BLU, R10.1, U$11.D
- new net N$16: D1.RED, R6.1, U$9.D
- new net N$17: CURRENT_POT.4, R19.1, R20.2
- new net N$18: CURRENT_POT.5, R20.1, R21.2
- new net N$19: CURRENT_POT.6, R21.1, R22.2
- new net N$20: CURRENT_POT.7, R22.1, R23.2
- new net N$21: CURRENT_POT.8, R23.1, R24.2
- new net N$22: CURRENT_POT.9, R24.1, R25.2
- new net N$23: R26.1, R45.1, TC_POT.1
- new net N$25: R26.2, R27.1, TC_POT.2
- new net N$26: R27.2, R28.2, TC_POT.3
- new net N$28: R28.1, R29.2, TC_POT.4
- new net N$29: R29.1, R30.2, TC_POT.5
- new net N$3: D5.C, U$3.D
- new net N$30: R30.1, R31.2, TC_POT.6
- new net N$31: R31.1, R32.2, TC_POT.7
- new net N$32: R32.1, R33.2, TC_POT.8
- new net N$33: R33.1, R34.2, TC_POT.9
- new net N$36: DRS_POT.2, R35.2, R36.1
- new net N$37: DRS_POT.3, R36.2, R37.2
- new net N$38: DRS_POT.1, R35.1, R46.1
- new net N$39: DRS_POT.4, R37.1, R38.2
- new net N$4: R3.1, S1.S
- new net N$40: DRS_POT.5, R38.1, R39.2
- new net N$41: DRS_POT.6, R39.1, R40.2
- new net N$42: DRS_POT.7, R40.1, R41.2
- new net N$43: DRS_POT.8, R41.1, R42.2
- new net N$44: DRS_POT.9, R42.1, R43.2
- new net N$5: D1.GRN, R8.1, U$12.D
- new net N$6: FUSE.2, L4.1
- new net N$8: D4.C, U$2.D
- new net PHONE_RX/U_TX: IC1PORTA_L.PA2, U$10.4
- new net PHONE_TX/U_RX: IC1PORTA_L.PA3, U$10.3
- new net PWR: FUSE.1, FUSE1.2, U$8.1
- new net TC_VALUE: IC1PORTA_L.PA7, TC_POT.COMMON
- net +3V3: now also D11.A
- net +5V: now also C2.+, D12.A, L4.2, R10.2, R44.2, R45.2, R46.2, R6.2, R8.2; no longer R4.2, R5.2, R9.2
- net BMS_LED: now also D5.A; no longer I/O1.5, U$3.D
- net BMS_LED_ON: no longer R6.2
- net BSPD_LED: now also D3.A; no longer I/O1.1, U$1.D
- net BSPD_LED_ON: no longer R10.2
- net CAN_H: now also U$8.4; no longer U$8.2
- net CAN_L: now also U$8.2; no longer U$8.4
- net GND: now also C2.-, CURRENT_POT.10, D1.C, DRS_POT.10, R13.1, R14.1, R25.1, R34.1, R43.1, S1.O, TC_POT.10, U$10.2, U$11.S, U$12.S, U$9.S; no longer I/O1.10, I/O1.2, I/O1.4, I/O1.6, I/O1.8, POWER.C, R10.1, R6.1, R8.1, U$5.S, U$7.3, U$7.4, U$9.2
- net IMD_LED: now also D4.A; no longer I/O1.3, U$2.D
- net IMD_LED_ON: no longer R8.2
- net N$7: now also CURRENT_POT.2, R15.2, R17.1; no longer I/O1.9
- net PHONE_POWER: now also FUSE1.1, U$10.1; no longer U$9.1
Other:
- note added: "GET RID OF THE SWITCHING REG FOR THE PHONE, WE WILL USE 5V FROM THE PHONE, WE WILL ALSO NOT NEED THE 12V, SO JUST ASSUME WE ARE GIVEN 5V. THEN GIVE A SMALL FUSE FOR THE MICRO AND A BIGGER FUSE FOR THE PHONE CHARGE, ALSO ATTACH A UART FOR THE PHONE"
- moved on the sheet: IC1AN_POWER, IC1RESET, R10, R3, R6, R8, U$1, U$2, U$3

Commit message: more tweaks
Connections:
- net PHONE_RX/U_TX: now also U$10.3; no longer U$10.4
- net PHONE_TX/U_RX: now also U$10.4; no longer U$10.3
Changed lines of the file:
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@@
 <net name="PHONE_TX/U_RX" class="0">
+<segment>
+<pinref part="IC1" gate="PORTA_L" pin="PA3"/>
+<wire x1="12.7" y1="-10.16" x2="7.62" y2="-10.16" width="0.1524" layer="91"/>
+<label x="7.62" y="-10.16" size="1.27" layer="95" rot="R180" xref="yes"/>
+</segment>
+<segment>
+<pinref part="U$10" gate="G$1" pin="4"/>
+<wire x1="-12.7" y1="43.18" x2="-2.54" y2="43.18" width="0.1524" layer="91"/>
+<label x="-2.54" y="43.18" size="1.27" layer="95" xref="yes"/>
+</segment>
+</net>
+<net name="PHONE_RX/U_TX" class="0">
+<segment>
+<pinref part="IC1" gate="PORTA_L" pin="PA2"/>
+<wire x1="12.7" y1="-7.62" x2="7.62" y2="-7.62" width="0.1524" layer="91"/>
+<label x="7.62" y="-7.62" size="1.27" layer="95" rot="R180" xref="yes"/>
+</segment>
 <segment>
 <pinref part="U$10" gate="G$1" pin="3"/>
@@
 <label x="-27.94" y="43.18" size="1.27" layer="95" rot="R180" xref="yes"/>
 </segment>
-<segment>
-<pinref part="IC1" gate="PORTA_L" pin="PA3"/>
-<wire x1="12.7" y1="-10.16" x2="7.62" y2="-10.16" width="0.1524" layer="91"/>
-<label x="7.62" y="-10.16" size="1.27" layer="95" rot="R180" xref="yes"/>
-</segment>
 </net>
-<net name="PHONE_RX/U_TX" class="0">
-<segment>
-<pinref part="U$10" gate="G$1" pin="4"/>
-<wire x1="-12.7" y1="43.18" x2="-2.54" y2="43.18" width="0.1524" layer="91"/>
-<label x="-2.54" y="43.18" size="1.27" layer="95" xref="yes"/>
-</segment>
-<segment>
-<pinref part="IC1" gate="PORTA_L" pin="PA2"/>
-<wire x1="12.7" y1="-7.62" x2="7.62" y2="-7.62" width="0.1524" layer="91"/>
-<label x="7.62" y="-7.62" size="1.27" layer="95" rot="R180" xref="yes"/>
-</segment>
-</net>

Commit message: v2 done
Parts:
- removed U$11, U$12: DMN2300U, Display_Custom:DMN2300U
- added C1, C3, C4, C6: 0.1u, rcl:C-EUC0805K
- added CUSTOM_POT: SWITCH_ROTARY_1X10KIT, Testing:SWITCH_ROTARY_1X10KIT
- added D6: DRS_BLUE, SparkFun-LED:LED-GREEN0603
- added D7: TC_BLUE, SparkFun-LED:LED-GREEN0603
- added Q1, Q2, Q6: DMP3099L-7, TRANS:DMP3099L-7
- added R4, R47, R48, R49, R5, R50, R51, R52, R53, R54, R55, R9: 10k, resistor:R-US_R0805
- added R56: 1k, resistor:R-US_R0805
- added R57, R58: 330, resistor:R-US_R0805
- added U$7: DMN2300U, Display_Custom:DMN2300U
- R1, R2, R7: value 10k -> 330
- R10: value 1k -> 85
- R13, R14: value (none) -> 330
- R6: value 1k -> 140
- R8: value 1k -> 90
Connections:
- removed net CAN_RX/STM_TX: IC1PORTA_H.PA12, U$6.RX
- removed net CAN_TX/STM_RX: IC1PORTA_H.PA11, U$6.TX
- removed net DASH_POWER_ON: IC1PORTB_L.PB2, U$9.G
- removed net DASH_PRE_DONE: IC1PORTB_H.PB11, U$12.G
- removed net DASH_PRE_STARTED: IC1PORTB_H.PB10, U$11.G
- new net CAN_RX: IC1PORTA_H.PA11, U$6.RX
- new net CAN_TX: IC1PORTA_H.PA12, U$6.TX
- new net CUSTOM_VALUE: CUSTOM_POT.COMMON, IC1PORTA_L.PA1
- new net DRS_: D6.A, R57.1
- new net DRS_LED: IC1PORTA_H.PA8, U$7.G
- new net N$1: Q6.D, R6.2
- new net N$24: Q1.D, R10.2
- new net N$27: Q2.D, R8.2
- new net N$34: CUSTOM_POT.2, R47.2, R48.1
- new net N$35: CUSTOM_POT.3, R48.2, R49.2
- new net N$45: CUSTOM_POT.4, R49.1, R50.2
- new net N$46: CUSTOM_POT.5, R50.1, R51.2
- new net N$47: CUSTOM_POT.6, R51.1, R52.2
- new net N$48: CUSTOM_POT.7, R52.1, R53.2
- new net N$49: CUSTOM_POT.8, R53.1, R54.2
- new net N$50: CUSTOM_POT.9, R54.1, R55.2
- new net N$51: CUSTOM_POT.1, R47.1, R56.1
- new net N$52: D6.C, U$7.D
- new net N$53: D7.C, U$9.D
- new net RGB_BLUE: IC1PORTB_H.PB10, Q1.G, R5.2
- new net RGB_GREEN: IC1PORTB_H.PB11, Q2.G, R9.2
- new net RGB_RED: IC1PORTB_L.PB2, Q6.G, R4.2
- new net TC_: D7.A, R58.1
- new net TC_LED: IC1PORTA_H.PA9, U$9.G
- net +3V3: now also C1.1, C3.1, C4.1, C6.1
- net +5V: now also Q1.S, Q2.S, Q6.S, R4.1, R5.1, R56.2, R57.2, R58.2, R9.1; no longer R10.2, R6.2, R8.2
- net DRS_VALUE: now also IC1PORTA_L.PA0; no longer IC1PORTB_L.PB0
- net GND: now also C1.2, C3.2, C4.2, C6.2, CUSTOM_POT.10, R55.1, U$7.S; no longer U$11.S, U$12.S
- net N$15: no longer U$11.D
- net N$16: no longer U$9.D
- net N$5: no longer U$12.D
Other:
- moved on the sheet: IC1AN_POWER, IC1PORTB_L, IC1RESET, U$9

Commit message: final revisions for 2
Connections:
- net GND: now also IC1PORTB_L.PB2
- net RGB_RED: now also IC1PORTB_L.PB0; no longer IC1PORTB_L.PB2
Changed lines of the file:
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@@
 <part name="P+11" library="supply1" deviceset="+5V" device=""/>
 <part name="D7" library="SparkFun-LED" deviceset="LED-GREEN" device="0603" value="TC_BLUE"/>
+<part name="GND20" library="supply1" deviceset="GND" device=""/>
+<part name="GND21" library="supply1" deviceset="GND" device=""/>
 </parts>
 <sheets>
@@
 <attribute name="NAME" x="-80.264" y="-80.772" size="1.778" layer="95" rot="R90"/>
 <attribute name="VALUE" x="-78.105" y="-80.772" size="1.778" layer="96" rot="R90"/>
+</instance>
+<instance part="GND20" gate="1" x="43.18" y="-119.38" smashed="yes">
+<attribute name="VALUE" x="40.64" y="-121.92" size="1.778" layer="96"/>
+</instance>
+<instance part="GND21" gate="1" x="60.96" y="-10.16" smashed="yes">
+<attribute name="VALUE" x="58.42" y="-12.7" size="1.778" layer="96"/>
 </instance>
 </instances>
@@
 <wire x1="-83.82" y1="-91.44" x2="-83.82" y2="-104.14" width="0.1524" layer="91"/>
 </segment>
+<segment>
+<pinref part="IC1" gate="PORTB_L" pin="PB2"/>
+<pinref part="GND21" gate="1" pin="GND"/>
+<wire x1="58.42" y1="-7.62" x2="60.96" y2="-7.62" width="0.1524" layer="91"/>
+</segment>
 </net>
 <net name="+3V3" class="0">
@@
 </segment>
 <segment>
-<pinref part="IC1" gate="PORTB_L" pin="PB2"/>
-<wire x1="58.42" y1="-7.62" x2="60.96" y2="-7.62" width="0.1524" layer="91"/>
-<label x="60.96" y="-7.62" size="1.27" layer="95" xref="yes"/>
-</segment>
-</net>
+<pinref part="IC1" gate="PORTB_L" pin="PB0"/>
+<wire x1="58.42" y1="-2.54" x2="60.96" y2="-2.54" width="0.1524" layer="91"/>
+<label x="60.96" y="-2.54" size="1.27" layer="95" xref="yes"/>
+</segment>
+</net>
