File: Boards/Tractive System/IFE_Shutdown_2019/Shutdown_2019_v1.1/Shutdown_2019_v1.1.sch (EAGLE design)
At the start: 195 parts, among them Q1 DMN6140L-7, Q10 DMN6140L-7, Q11 DMP3099L-7, Q12 IRLML6346PBF, Q13 IRLML6346PBF, Q14 IRLML6346PBF, Q15 DMP3099L-7, Q16 DMN6140L-7, Q17 IRLML6346PBF, Q18 DMN6140L-7, Q2 DMN6140L-7, Q20 DMN6140L-7, Q21 DMN6140L-7, Q3 DMN6140L-7, Q4 DMN6140L-7, Q5 DMN6140L-7, Q6 DMP3099L-7, Q7 DMN6140L-7, Q9 DMN6140L-7, U1 STM32F103CBT6, U2 STM32F103CBT6

Commit message: Still working on 1.1
Parts:
- removed BUZZER: PKMCS0909E4000, MURATA:PKMCS0909E4000
- added U$6: MAS806Q, MALLORY:MAS806Q
Connections:
- net +12V: now also U$6.A; no longer BUZZER.A
- net N$4: now also U$6.B; no longer BUZZER.B
Changed lines of the file:
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@@
 <?xml version="1.0" encoding="utf-8"?>
 <!DOCTYPE eagle SYSTEM "eagle.dtd">
-<eagle version="9.2.2">
+<eagle version="9.1.2">
 <drawing>
 <settings>
@@
 <part name="P+46" library="supply1" deviceset="+5V" device=""/>
 <part name="C39" library="resistor" library_urn="urn:adsk.eagle:library:348" deviceset="C-US" device="C0603" package3d_urn="urn:adsk.eagle:package:26138/1" value="0.1u"/>
-<part name="BUZZER" library="MURATA" deviceset="PKMCS0909E4000" device=""/>
 <part name="P+4" library="supply1" library_urn="urn:adsk.eagle:library:371" deviceset="+12V" device=""/>
 <part name="AGND1" library="supply1" library_urn="urn:adsk.eagle:library:371" deviceset="AGND" device=""/>
@@
 <part name="U$2" library="KEMET" deviceset="EC2" device=""/>
 <part name="U$3" library="KEMET" deviceset="EC2" device=""/>
+<part name="U$6" library="MALLORY" deviceset="MAS806Q" device=""/>
 </parts>
 <sheets>
@@
 <attribute name="VALUE" x="190.5" y="111.76" size="1.778" layer="96"/>
 </instance>
-<instance part="BUZZER" gate="G$1" x="193.04" y="139.7" smashed="yes"/>
 <instance part="P+4" gate="1" x="193.04" y="147.32" smashed="yes">
 <attribute name="VALUE" x="190.5" y="142.24" size="1.778" layer="96" rot="R90"/>
 </instance>
+<instance part="U$6" gate="G$1" x="193.04" y="139.7"/>
 </instances>
 <busses>
@@
 <net name="N$4" class="0">
 <segment>
-<pinref part="BUZZER" gate="G$1" pin="B"/>
 <pinref part="Q4" gate="G$1" pin="D"/>
 <wire x1="193.04" y1="137.16" x2="193.04" y2="134.62" width="0.1524" layer="91"/>
+<pinref part="U$6" gate="G$1" pin="B"/>
 </segment>
 </net>
 <net name="+12V" class="3">
 <segment>
-<pinref part="BUZZER" gate="G$1" pin="A"/>
 <wire x1="193.04" y1="142.24" x2="193.04" y2="144.78" width="0.1524" layer="91"/>
 <pinref part="P+4" gate="1" pin="+12V"/>
+<pinref part="U$6" gate="G$1" pin="A"/>
 </segment>
 </net>

Commit message: Finished pre review Safety V1.1
Parts:
- removed CURRENT_SENSOR_SUPPLY, PWR: MINIFIT_JR_5566-02, Display_Custom:MINIFIT_JR_5566-02
- removed DRIVERS, FAULT_INPUT, HALL_SENSE, THROTTLE, TSAL_EN: MINIFIT_JR_5566-04, Display_Custom:MINIFIT_JR_5566-04
- removed Q17: IRLML6346PBF, TRANS:IRLML6346PBF
- removed R6: 3.6k, rcl:R-US_R0603
- added C40, C41: 0.001u, rcl:C-USC0805
- added C42, C43, C44, C45, C46: 0.1u, resistor:C-USC0603
- added CURRENT_SENSE_SUPPLY, POWER, POWER_ANALOG, SOFT_FAULT_STAT: 505575-02, MOLEX:505575-02
- added FAULT_IN, LIGHTING, THROTTLE_TC: 505575-05, MOLEX:505575-05
- added FAULT_STAT: 505575-03, MOLEX:505575-03
- added HALL_SENSOR_INPUT: 505575-04, MOLEX:505575-04
- added Q8: DMN6140L-7, TRANS:DMN6140L-7
- added R10, R78: 10, rcl:R-US_R0603
- added R45, R75, R79, R80: 10k, rcl:R-US_R0603
- added R76, R81: 15k, rcl:R-US_R0603
- added R77, R82: 1k, rcl:R-US_R0603
- added R83: 10k, resistor:R-US_R0603
- added U$13, U$15: LMV321L, STM:LMV321L
- added U$14, U$19: BZT52C5V6, DIODES_INC:BZT52C
- added U$27: SN74LVC1G08, TEXAS_INSTRUMENTS:SN74LVC1G08
- added U$28: CD4072BM96, TEXAS_INSTRUMENTS:CD4072B
- added U$30, U$31: TS881, STM:TS881
- AIR, CAN, ENABLE: value MINIFIT_JR_5566-02 -> 505575-02; device Display_Custom:MINIFIT_JR_5566-02 -> MOLEX:505575-02
- Q13: value IRLML6346PBF -> DMN6140L-7; device TRANS:IRLML6346PBF -> TRANS:DMN6140L-7
- R3: value 3.6k -> 10k; device rcl:R-US_R0603 -> resistor:R-US_R0603
- U$7: value DNBT8105 -> SN74LVC1G04DBVR; device DIODES_INC:DNBT8105 -> Display_Custom:SN74LVC1G04DBVR
- U$8: value DNBT8105 -> 0805_INDUCTOR; device DIODES_INC:DNBT8105 -> Display_Custom:0805_INDUCTOR
Connections:
- removed net BSPD_OC: Q17.G, U$17.OUT
- removed net BSPD_SC: Q14.G, U$16.OUT
- removed net N$15: R3.2, U$8.B
- removed net N$16: R6.2, U$7.B
- removed net TSAL_HV_EN: R3.1, U1.PB11
- removed net TSAL_LV_EN: R6.1, U1.PB12
- new net APPS_STAT: SOFT_FAULT_STAT.1
- new net BRAKE_POS: R10.1, THROTTLE_TC.5
- new net BRAKE_POS_F: R75.2, U$13.-IN, U$13.OUT
- new net BRAKE_POS_F_3_3: R75.1, R76.2, U1.PA1
- new net BSPD_BP_OC: U$28.A0, U$31.OUT
- new net BSPD_BP_SC: U$28.B0, U$30.OUT
- new net BSPD_COND: Q12.G, R83.2, U$27.Y
- new net BSPD_CS_OC: U$17.OUT, U$28.C0
- new net BSPD_CS_SC: U$16.OUT, U$28.D0
- new net BSPD_SENSOR_FAULT: Q14.G, U$28.Y0
- new net BTSF_STAT: SOFT_FAULT_STAT.2
- new net N$22: R78.2, R79.1, R82.1, U$19.C
- new net N$23: C41.1, R79.2, U$15.+IN
- new net N$5: R10.2, R45.1, R77.1, U$14.C
- new net N$7: C40.1, R45.2, U$13.+IN
- new net STEERING_POS: R78.1, THROTTLE_TC.4
- new net STEERING_POS_F: R80.2, U$15.-IN, U$15.OUT
- new net STEERING_POS_F_3_3: R80.1, R81.2, U1.PA2
- net +3V3: now also U$7.V+
- net +5V: now also C42.1, C43.1, C44.1, C45.1, C46.1, CURRENT_SENSE_SUPPLY.1, R77.2, R82.2, U$13.VDD, U$15.VDD, U$27.VDD, U$28.VDD, U$30.VDD, U$31.VDD; no longer CURRENT_SENSOR_SUPPLY.1, TSAL_EN.1
- net AGND: now also POWER_ANALOG.2, U$8.1
- net AIR_IN: now also AIR.2; no longer AIR.1
- net AIR_OUT: now also AIR.1; no longer AIR.2
- net ANALOG_5V: now also POWER_ANALOG.1
- net BRAKE_LIGHT-: now also LIGHTING.4; no longer DRIVERS.1
- net BRAKE_PRESSURE: now also FAULT_IN.4; no longer FAULT_INPUT.4
- net BRAKE_PRESSURE_F: now also U$30.-IN, U$31.+IN
- net BSPD_BRAKE_COND: now also U$27.B; no longer Q13.G
- net BSPD_CURR_COND: now also U$27.A; no longer Q12.G
- net CURRENT_SENSE: now also FAULT_IN.5; no longer FAULT_INPUT.2
- net ENABLE_IN: now also ENABLE.2; no longer ENABLE.1
- net ENABLE_OUT: now also ENABLE.1; no longer ENABLE.2
- net FAULT_BMS: now also FAULT_IN.3; no longer FAULT_INPUT.1
- net FAULT_BMS_STAT: now also FAULT_STAT.2
- net FAULT_BMS_STATUS_3_3: now also U1.PB11; no longer U1.PA2
- net FAULT_BSPD: no longer Q17.D
- net FAULT_BSPD_STAT: now also FAULT_STAT.1
- net FAULT_IMD: now also FAULT_IN.2; no longer FAULT_INPUT.3
- net FAULT_IMD_STAT: now also FAULT_STAT.3
- net FAULT_RESET: now also FAULT_IN.1; no longer TSAL_EN.4
- net GND: now also C40.2, C41.2, C42.2, C43.2, C44.2, C45.2, C46.2, CURRENT_SENSE_SUPPLY.2, POWER.2, Q12.S, Q8.S, R3.1, R76.1, R81.1, R83.1, U$13.GND, U$14.A, U$15.GND, U$19.A, U$27.GND, U$28.GND, U$30.GND, U$31.GND, U$7.GND, U$8.2; no longer CURRENT_SENSOR_SUPPLY.2, PWR.2, Q17.S, TSAL_EN.3, U$7.E, U$8.E
- net HALL_FL: now also HALL_SENSOR_INPUT.1; no longer HALL_SENSE.1
- net HALL_FR: now also HALL_SENSOR_INPUT.2; no longer HALL_SENSE.3
- net HALL_RL: now also HALL_SENSOR_INPUT.3; no longer HALL_SENSE.2
- net HALL_RR: now also HALL_SENSOR_INPUT.4; no longer HALL_SENSE.4
- net HV_CONNECTED_3_3: now also Q8.G, U$7.A
- net N$9: now also Q13.G, R3.2, U$7.Y; no longer Q12.S, Q13.D
- net OC_TH: now also U$31.-IN
- net PRECHARGE_COMPLETE: now also LIGHTING.5; no longer THROTTLE.3
- net PWR: now also POWER.1; no longer PWR.1
- net SC_TH: now also U$30.+IN
- net THROTTLE_A: now also THROTTLE_TC.1; no longer THROTTLE.1
- net THROTTLE_B: now also THROTTLE_TC.2; no longer THROTTLE.2
- net THROTTLE_OUT: now also THROTTLE_TC.3; no longer THROTTLE.4
- net TSAL_EN: now also LIGHTING.1; no longer TSAL_EN.2
- net TSAL_HV-: now also LIGHTING.3, Q8.D; no longer DRIVERS.4, U$8.C
- net TSAL_LV-: now also LIGHTING.2, Q13.D; no longer DRIVERS.2, U$7.C
Other:
- moved on the sheet: C32, Q10, Q12, Q14, Q7, R23, R3, R5, R55, R56, R74, U$21

Commit message: Ready to route
Connections:
- net AGND: now also C21.2
- net BRAKE_POS: now also THROTTLE_TC.4; no longer THROTTLE_TC.5
- net CANH: now also CAN.1; no longer CAN.2
- net CANL: now also CAN.2; no longer CAN.1
- net GND: no longer C21.2
- net STEERING_POS: now also THROTTLE_TC.3; no longer THROTTLE_TC.4
- net THROTTLE_OUT: now also THROTTLE_TC.5; no longer THROTTLE_TC.3
Changed lines of the file:
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@@
 <part name="U$18" library="STM" deviceset="LMV321L" device=""/>
 <part name="C21" library="rcl" library_urn="urn:adsk.eagle:library:334" deviceset="C-US" device="C0603" package3d_urn="urn:adsk.eagle:package:23616/2" value="1u"/>
-<part name="GND9" library="supply1" library_urn="urn:adsk.eagle:library:371" deviceset="GND" device=""/>
 <part name="U$22" library="STM" deviceset="LMV321L" device=""/>
 <part name="U$23" library="STM" deviceset="LMV321L" device=""/>
@@
 <part name="AGND5" library="supply1" library_urn="urn:adsk.eagle:library:371" deviceset="AGND" device=""/>
 <part name="GND8" library="supply1" library_urn="urn:adsk.eagle:library:371" deviceset="GND" device=""/>
+<part name="AGND6" library="supply1" library_urn="urn:adsk.eagle:library:371" deviceset="AGND" device=""/>
 </parts>
 <sheets>
@@
 </busses>
 <nets>
-<net name="CANL" class="0">
-<segment>
-<pinref part="CAN" gate="G$1" pin="1"/>
-<wire x1="-147.32" y1="104.14" x2="-144.78" y2="104.14" width="0.1524" layer="91"/>
-<label x="-144.78" y="104.14" size="1.27" layer="95" xref="yes"/>
-</segment>
-</net>
 <net name="GND" class="0">
 <segment>
@@
 <net name="CANH" class="0">
 <segment>
-<pinref part="CAN" gate="G$1" pin="2"/>
-<wire x1="-147.32" y1="101.6" x2="-144.78" y2="101.6" width="0.1524" layer="91"/>
-<label x="-144.78" y="101.6" size="1.27" layer="95" xref="yes"/>
+<pinref part="CAN" gate="G$1" pin="1"/>
+<wire x1="-147.32" y1="104.14" x2="-144.78" y2="104.14" width="0.1524" layer="91"/>
+<label x="-144.78" y="104.14" size="1.27" layer="95" xref="yes"/>
 </segment>
 </net>
@@
 <net name="THROTTLE_OUT" class="0">
 <segment>
-<pinref part="THROTTLE_TC" gate="G$1" pin="3"/>
-<wire x1="-116.84" y1="104.14" x2="-114.3" y2="104.14" width="0.1524" layer="91"/>
-<label x="-114.3" y="104.14" size="1.27" layer="95" xref="yes"/>
+<pinref part="THROTTLE_TC" gate="G$1" pin="5"/>
+<wire x1="-116.84" y1="99.06" x2="-114.3" y2="99.06" width="0.1524" layer="91"/>
+<label x="-114.3" y="99.06" size="1.27" layer="95" xref="yes"/>
 </segment>
 </net>
 <net name="STEERING_POS" class="0">
 <segment>
-<pinref part="THROTTLE_TC" gate="G$1" pin="4"/>
-<wire x1="-116.84" y1="101.6" x2="-114.3" y2="101.6" width="0.1524" layer="91"/>
-<label x="-114.3" y="101.6" size="1.27" layer="95" xref="yes"/>
-</segment>
-<segment>
 <pinref part="R78" gate="G$1" pin="1"/>
 <wire x1="134.62" y1="5.08" x2="132.08" y2="5.08" width="0.1524" layer="91"/>
 <label x="132.08" y="5.08" size="1.27" layer="95" rot="R180" xref="yes"/>
 </segment>
-</net>
-<net name="BRAKE_POS" class="0">
 <segment>
-<pinref part="THROTTLE_TC" gate="G$1" pin="5"/>
-<wire x1="-116.84" y1="99.06" x2="-114.3" y2="99.06" width="0.1524" layer="91"/>
-<label x="-114.3" y="99.06" size="1.27" layer="95" xref="yes"/>
+<pinref part="THROTTLE_TC" gate="G$1" pin="3"/>
+<wire x1="-116.84" y1="104.14" x2="-114.3" y2="104.14" width="0.1524" layer="91"/>
+<label x="-114.3" y="104.14" size="1.27" layer="95" xref="yes"/>
 </segment>
+</net>
+<net name="BRAKE_POS" class="0">
 <segment>
 <pinref part="R10" gate="G$1" pin="1"/>
@@
 <label x="0" y="7.62" size="1.27" layer="95" rot="R180" xref="yes"/>
 </segment>
+<segment>
+<pinref part="THROTTLE_TC" gate="G$1" pin="4"/>
+<wire x1="-116.84" y1="101.6" x2="-114.3" y2="101.6" width="0.1524" layer="91"/>
+<label x="-114.3" y="101.6" size="1.27" layer="95" xref="yes"/>
+</segment>
 </net>
 <net name="APPS_STAT" class="0">
@@
 </segment>
 </net>
+<net name="CANL" class="0">
+<segment>
+<pinref part="CAN" gate="G$1" pin="2"/>
+<wire x1="-147.32" y1="101.6" x2="-144.78" y2="101.6" width="0.1524" layer="91"/>
+<label x="-144.78" y="101.6" size="1.27" layer="95" xref="yes"/>
+</segment>
+</net>
 </nets>
 </sheet>
@@
 <attribute name="VALUE" x="315.976" y="201.549" size="1.778" layer="96"/>
 </instance>
-<instance part="GND9" gate="1" x="314.96" y="195.58" smashed="yes">
-<attribute name="VALUE" x="312.42" y="193.04" size="1.778" layer="96"/>
-</instance>
 <instance part="R47" gate="G$1" x="246.38" y="198.12" smashed="yes" rot="R270">
 <attribute name="NAME" x="247.8786" y="201.93" size="1.778" layer="95" rot="R270"/>
@@
 <attribute name="VALUE" x="289.56" y="175.26" size="1.778" layer="96" rot="R90"/>
 </instance>
+<instance part="AGND6" gate="VR1" x="314.96" y="195.58" smashed="yes">
+<attribute name="VALUE" x="312.42" y="190.5" size="1.778" layer="96" rot="R90"/>
+</instance>
 </instances>
 <busses>
@@
 </segment>
 <segment>
-<pinref part="C21" gate="G$1" pin="2"/>
-<pinref part="GND9" gate="1" pin="GND"/>
-<wire x1="314.96" y1="200.66" x2="314.96" y2="198.12" width="0.1524" layer="91"/>
-</segment>
-<segment>
 <pinref part="C33" gate="G$1" pin="2"/>
 <wire x1="266.7" y1="152.4" x2="266.7" y2="149.86" width="0.1524" layer="91"/>
@@
 <pinref part="AGND3" gate="VR1" pin="AGND"/>
 </segment>
+<segment>
+<pinref part="C21" gate="G$1" pin="2"/>
+<wire x1="314.96" y1="200.66" x2="314.96" y2="198.12" width="0.1524" layer="91"/>
+<pinref part="AGND6" gate="VR1" pin="AGND"/>
+</segment>
 </net>

Commit message: finished safety v1.1 layout
Connections:
- removed net APPS_STAT: SOFT_FAULT_STAT.1
- removed net BTSF_STAT: SOFT_FAULT_STAT.2
- net APPS_EN: now also SOFT_FAULT_STAT.1
- net BSPD_BP_SC: now also U$28.C0; no longer U$28.B0
- net BSPD_CS_OC: now also U$28.B0; no longer U$28.C0
- net BTSF_EN: now also SOFT_FAULT_STAT.2
Changed lines of the file:
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@@
 </segment>
 <segment>
-<pinref part="U$28" gate="G$1" pin="C0"/>
-<wire x1="139.7" y1="129.54" x2="137.16" y2="129.54" width="0.1524" layer="91"/>
-<label x="137.16" y="129.54" size="1.27" layer="95" rot="R180" xref="yes"/>
+<pinref part="U$28" gate="G$1" pin="B0"/>
+<wire x1="139.7" y1="132.08" x2="137.16" y2="132.08" width="0.1524" layer="91"/>
+<label x="137.16" y="132.08" size="1.27" layer="95" rot="R180" xref="yes"/>
 </segment>
 </net>
@@
 </segment>
 <segment>
-<pinref part="U$28" gate="G$1" pin="B0"/>
-<wire x1="139.7" y1="132.08" x2="137.16" y2="132.08" width="0.1524" layer="91"/>
-<label x="137.16" y="132.08" size="1.27" layer="95" rot="R180" xref="yes"/>
+<pinref part="U$28" gate="G$1" pin="C0"/>
+<wire x1="139.7" y1="129.54" x2="137.16" y2="129.54" width="0.1524" layer="91"/>
+<label x="137.16" y="129.54" size="1.27" layer="95" rot="R180" xref="yes"/>
 </segment>
 </net>
@@
 </segment>
 </net>
-<net name="APPS_STAT" class="0">
+<net name="APPS_EN" class="0">
 <segment>
 <pinref part="SOFT_FAULT_STAT" gate="G$1" pin="1"/>
@@
 </segment>
 </net>
-<net name="BTSF_STAT" class="0">
+<net name="BTSF_EN" class="0">
 <segment>
 <pinref part="SOFT_FAULT_STAT" gate="G$1" pin="2"/>
