File: Boards/Tractive System/IFE_Precharge_2019/Precharge_M2019_V1.1.sch (EAGLE design)
At the start: 20 parts

Commit message: Precharge 1.2 finished, added .gitignore
Parts:
- removed RELAY: MINIFIT_JR_5566-02, Display_Custom:MINIFIT_JR_5566-02
- removed U$2: MINIFIT_JR_5566-04, Display_Custom:MINIFIT_JR_5566-04
- added H1, H2, H3, H4: MOUNT-PAD-ROUND3.0, holes:MOUNT-PAD-ROUND3.0
- added U$7: 505575-02, MOLEX:505575-02
- added U$8: 505575-03, MOLEX:505575-03
Connections:
- removed net N$4: D2.A, RELAY.1, U$3.D
- new net RELAY-: D2.A, U$3.D, U$7.2
- net GND: now also H1.MOUNT, H2.MOUNT, H3.MOUNT, H4.MOUNT, U$8.1; no longer U$2.4
- net PRECHARGE_COMPLETE: now also U$8.2; no longer U$2.1
- net V+: now also U$7.1, U$8.3; no longer RELAY.2, U$2.3
