File: Boards/Strain_gauge/strain.sch (EAGLE design)
At the start: 69 parts, among them U1 ADS1262IPW, U2 STM32F103CBT6

Commit message: Rushed the fuck out of the ADS1262 board, but here it is
Parts:
- removed IC1: (no value), v-reg-3:LM317TL
- removed R21, R22: 750, rcl:R-US_R0805
- added IC2: 317EMP, linear:317EMP
Connections:
- removed net APPS_EN: U2.PB4
- removed net BRAKE_LIGHT_EN: U2.PB13
- removed net BRAKE_PRESSURE_F_3_3: U2.PA0-WKUP
- removed net BTSF_EN: U2.PB5
- removed net CAN_RX: U2.PA11
- removed net CAN_STBY: U2.PA10
- removed net CAN_TX: U2.PA12
- removed net FAULT_BMS_STATUS_3_3: U2.PA2
- removed net FAULT_BSPD_STATUS_3_3: U2.PB14
- removed net FAULT_IMD_STATUS_3_3: U2.PA3
- removed net HV_CONNECTED_3_3: U2.PB10
- removed net N$27: IC1.ADJ, R21.1, R22.1
- removed net PRECHARGE_COMPLETE_3_3: U2.PB6
- removed net RTDS_EN: U2.PB3
- removed net RTD_EN: U2.PB8
- removed net SPI1_MISO: U2.PA6
- removed net SPI1_MOSI: U2.PA7
- removed net SPI1_NSS: U2.PA4
- removed net SPI1_SCK: U2.PA5
- removed net THROTTLE_A_F_3_3: U2.PB0
- removed net THROTTLE_B_F_3_3: U2.PB1
- removed net TSAL_HV_EN: U2.PB11
- removed net TSAL_LV_EN: U2.PB12
- new net RX: SV1.10, U2.PA9
- new net TX: SV1.8, U2.PA10
- net +3V3: now also IC2.VO; no longer IC1.OUT, R21.2, SV1.1, SV1.17
- net ADC_0: now also U2.PB0
- net ADC_1: now also U2.PB1
- net ADC_2: now also U2.PB3
- net ADC_3: now also U2.PB4
- net ADC_4: now also U2.PB5
- net ADC_5: now also U2.PB6
- net ADC_6: now also U2.PB7
- net ADC_7: now also U2.PB8
- net ADC_8: now also U2.PB9
- net CS: no longer SV1.13
- net DIN: no longer SV1.16
- net DOUT: no longer SV1.18
- net DRDY: no longer SV1.22
- net GND: now also IC2.ADJ; no longer R22.2, SV1.14, SV1.20, SV1.25, SV1.30, SV1.34, SV1.39, SV1.9
- net IN_F: now also IC2.VI; no longer IC1.IN
- net RESET: no longer SV1.36
- net SCLK: no longer SV1.15
- net START: no longer SV1.11
